Commit message: Updated IMU sensor

File: src/voyager_description/urdf/voyager.urdf.xacro (robot description, xacro)
@@ -201,3 +201,23 @@
         <limit lower="-0.5" upper="0.5" effort="0.5" velocity="0.8"/>
     </joint>
+    <!-- IMU link -->
+    <link name="imu_link">
+        <inertial>
+            <origin xyz="0.0 0.0 0.0" rpy="0.0 0.0 0.0"/>
+            <mass value="0.005"/>
+            <inertia ixx="8.333333333333334e-08" ixy="0.0" ixz="0.0" iyy="8.333333333333334e-08" iyz="0.0" izz="8.333333333333334e-08"/>
+        </inertial>
+        <visual name="">
+            <origin xyz="0.0 0.0 0.0" rpy="0.0 0.0 0.0"/>
+            <geometry>
+                <box size="0.01 0.01 0.01"/>
+            </geometry>
+        </visual>
+    </link>
+    <joint name="imu_joint" type="fixed">
+        <origin xyz="0.0 0.0 0.015" rpy="0.0 0.0 0.0"/>
+        <parent link="base_link"/>
+        <child link="imu_link"/>
+        <axis xyz="0.0 0.0 0.0"/>
+    </joint>
 </robot>

File: src/voyager_description/urdf/voyager_gazebo.xacro (robot description, xacro)
@@ -79,3 +79,22 @@
         </plugin>
     </gazebo>
+      <!-- IMU -->
+  <gazebo reference="imu_link">
+    <gravity>true</gravity>
+    <sensor name="imu_sensor" type="imu">
+      <always_on>true</always_on>
+      <update_rate>10</update_rate>
+      <visualize>true</visualize>
+      <plugin filename="libgazebo_ros_imu_sensor.so" name="imu">
+        <bodyName>imu_link</bodyName>
+        <updateRateHZ>10.0</updateRateHZ>
+        <gaussianNoise>0.0</gaussianNoise>
+        <xyzOffset>0 0 0</xyzOffset>
+        <rpyOffset>0 0 0</rpyOffset>
+        <frameName>imu_link</frameName>
+        <initialOrientationAsReference>false</initialOrientationAsReference>
+      </plugin>
+      <pose>0 0 0 0 0 0</pose>
+    </sensor>
+  </gazebo>
 </robot>
